File: shield/shield.kicad_pcb (KiCad board)
At the start: 4 copper layers, 74.5 x 120 mm, 73 parts, among them CON1 MSATA-PCIE_MINI-CARD-MM60-52B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, J1 Conn_02x12_Top_Bottom, J2 SIM_Card, K1 G5Q-1A, K2 G5Q-1A, K3 G5Q-1A, Q1 Q_NPN_BEC, Q2 Q_NPN_BEC, Q3 Q_NPN_BEC, U1 orange_pi_zero, U2 MCP25625-x-SS, U3 OKI-78SR-5_1.5-W36-C, U4 MCP25625-x-SS, U5 LD1085D2M33R, Y1 M8AIG-16-12-2T3, Y2 M8AIG-16-12-2T3

Commit message: m
Parts:
- added C27: 4.7uF, Capacitor_SMD:C_0603_1608Metric, F.Cu at (47.2, 77.2)
- added C28: 0.1uF, Capacitor_SMD:C_0603_1608Metric, F.Cu at (47.2, 73.8)
- added C29: 0.1uF, Capacitor_SMD:C_0603_1608Metric, F.Cu at (45.0, 70.7)
- added G***: LOGO, aep:artanis, B.Cu at (39.0, 53.0)
- added R21: 4.7K, Resistor_SMD:R_0603_1608Metric, F.Cu at (43.8, 72.3)
- added R22: 4.7K, Resistor_SMD:R_0603_1608Metric, F.Cu at (39.7, 73.2)
- added REF**: OSHW-Logo2_7.3x6mm_SilkScreen, Symbol:OSHW-Logo2_7.3x6mm_SilkScreen, B.Cu at (31.0, 61.0)
- added REF**: ESD-Logo_6.6x6mm_SilkScreen, Symbol:ESD-Logo_6.6x6mm_SilkScreen, B.Cu at (40.0, 60.8)
- added REF**: WEEE-Logo_4.2x6mm_SilkScreen, Symbol:WEEE-Logo_4.2x6mm_SilkScreen, B.Cu at (47.0, 61.0)
- added TP1: SA0, OLIMEX_TestPoints-FP:TP_SMD, F.Cu at (39.7, 75.7)
- added U7: MMA8452Q, Silicon-Custom:QFN-16, F.Cu at (43.5, 75.6)
- moved FID1 60.9 mm to (72.7, 122.0)
Connections:
- U1 pad 101: (no net) -> 3.3V
- U1 pad 103: (no net) -> TWI0_SDA
- U1 pad 105: (no net) -> TWI0_SCK
- U1 pad 111: (no net) -> IMU_INT2
- U1 pad 112: (no net) -> IMU_INT1
Routing:
- net 3.3V: track 104.3 -> 205.8 mm
- net 5V: track 197.2 -> 223.7 mm
- net IMU_INT2: track 0.00 -> 24.5 mm
- net IMU_INT1: track 0.00 -> 23.9 mm
- net TWI0_SCK: track 0.00 -> 23.2 mm, vias 0 -> 1
- net GND: track 202.6 -> 224.0 mm, vias 97 -> 314
- net TWI0_SDA: track 0.00 -> 20.1 mm
- net USB2+: track 82.9 -> 77.5 mm
- net Net-(C29-Pad1): track 0.00 -> 3.67 mm
- net Net-(TP1-Pad1): track 0.00 -> 2.57 mm
- net /c2_P: track 97.3 -> 98.1 mm
- net /c2_N: track 100.1 -> 100.9 mm
- net VCC3V3: vias 0 -> 3
- added copper zone on Supply.Cu, net 3.3V
- added copper zone on Supply.Cu, net VCC3V3
Other:
- net class Default: clearance 0.2 -> 0.1778
- rule trace_clearance: 0.2 -> 0.1778
- board text added: "prototype not for sale v 0.2 | 2019 | aep"
