File: shield/shield.sch (KiCad schematic (older format))
At the start: 79 parts, among them CON1 MSATA-PCIE_MINI-CARD-MM60-52B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, J1 Conn_02x12_Top_Bottom, J2 SIM_Card, K1 G5Q-1A, K2 G5Q-1A, K3 G5Q-1A, Q1 Q_NPN_BEC, Q2 Q_NPN_BEC, Q3 Q_NPN_BEC, Q4 Q_NPN_BEC, U1 orange_pi_zero, U2 MCP25625-x-SS, U3 OKI-78SR-5_1.5-W36-C, U4 MCP25625-x-SS, U5 LD1085D2M33R, U6 ASSR-1218, Y1 M8AIG-16-12-2T3, Y2 M8AIG-16-12-2T3

Commit message: m
Parts:
- removed Q4: Q_NPN_BEC, Silicon-Standard:SOT23-3, symbol Device:Q_NPN_BEC
- removed R17: 1K, Resistor_SMD:R_0603_1608Metric, symbol Device:R
- removed R18, R20: 10K, Resistor_SMD:R_0603_1608Metric, symbol Device:R
- removed R19: 100, Resistor_SMD:R_0603_1608Metric, symbol Device:R
- removed U6: ASSR-1218, Package_SO:SO-4_4.4x4.3mm_P2.54mm, symbol Relay_SolidState:ASSR-1218
- added C27: 4.7uF, Capacitor_SMD:C_0603_1608Metric, symbol Device:C
- added C28, C29: 0.1uF, Capacitor_SMD:C_0603_1608Metric, symbol Device:C
- added R21, R22: 4.7K, Resistor_SMD:R_0603_1608Metric, symbol Device:R
- added TP1: SA0, OLIMEX_TestPoints-FP:TP_SMD, symbol Connector:TestPoint_Alt
- added U7: MMA8452Q, QFN-16, symbol SparkFun-Sensors:MMA8452Q
Connections:
- net 3.3V: now also U1.101 (3.3V), C27.1, C28.1, R21.2, R22.2, U7.1 (VDDIO), U7.14 (VDD)
- net GND: now also C27.2, C28.2, C29.2, U7.10 (GND), U7.12 (GND), U7.5 (GND)
- net TWI0_SDA: now reaches U1.103 (TWI0_SDA_/_PA12)
- net TWI0_SDA: now also R22.1, U7.6 (SDA)
- net TWI0_SCK: now reaches U1.105 (TWI0_SCK_/_PA11)
- net TWI0_SCK: now also R21.1, U7.4 (SCL)
- net IMU_INT2: now reaches U1.111 (UART2_RX_/_PA01)
- net IMU_INT2: now also U7.9 (INT2)
- net IMU_INT1: now reaches U1.112 (SIM_CLK/PA_EINT7_/_PA07)
- net IMU_INT1: now also U7.11 (INT1)
- new net: C29.1, U7.2 (BYP)
- new net: TP1.1, U7.7 (SA0)
Other:
- note removed: "TODO\nVERIFY IRQ SETUP"
