File: base/0.2.kicad_pcb (KiCad board)
At the start: 4 copper layers, 74.5 x 120 mm, 84 parts, among them CON1 MSATA-PCIE_MINI-CARD-MM60-52B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, J1 Conn_02x12_Top_Bottom, J2 SIM_Card, K1 G5Q-1A, K2 G5Q-1A, K3 G5Q-1A, Q1 Q_NPN_BEC, Q2 Q_NPN_BEC, Q3 Q_NPN_BEC, U1 orange_pi_zero, U2 MCP25625-x-SS, U3 OKI-78SR-5_1.5-W36-C, U4 MCP25625-x-SS, U5 LD1085D2M33R, U7 MMA8452Q, Y1 M8AIG-16-12-2T3, Y2 M8AIG-16-12-2T3

Commit message: m
Parts:
- removed the G*** at (39.0, 53.0)
- added G***: LOGO, aep:devguard, F.Cu at (37.5, 51.5)
- added G***: LOGO, aep:devguard, B.Cu at (37.5, 50.0)
- added G***: LOGO, aep:devguard, F.Cu at (43.5, 52.5)
- moved FID1 16.0 mm to (72.7, 106.0)
- moved C19 3.00 mm to (5.40, 47.0)
- moved C20 3.00 mm to (5.40, 50.3)
- moved CON1 3.00 mm to (14.5, 52.0)
- moved REF** 2.80 mm to (37.5, 59.5)
- moved REF** 2.50 mm to (45.0, 59.5)
- moved REF** 2.50 mm to (29.0, 59.5)
Connections:
- R2 pad 1: Net-(R2-Pad1) -> (no net)
- R4 pad 1: Net-(R4-Pad1) -> (no net)
Routing:
- net 5V: track 223.7 -> 155.6 mm
- net GND: track 224.0 -> 214.1 mm, vias 314 -> 329
- net USB2+: track 77.5 -> 85.9 mm
- net Net-(CON1-Pad10): track 51.6 -> 55.4 mm
- net USB2-: track 82.7 -> 85.7 mm
- net Net-(CON1-Pad16): track 59.4 -> 61.2 mm
- net Net-(CON1-Pad12): track 48.9 -> 50.6 mm
- net Net-(CON1-Pad44): track 22.2 -> 21.0 mm
- net Net-(CON1-Pad42): track 21.3 -> 20.0 mm
- net Net-(CON1-Pad46): track 24.1 -> 22.9 mm
- net Net-(C25-Pad1): track 66.2 -> 65.1 mm
- net VCC3V3: track 168.4 -> 169.5 mm
- net (no net): vias 0 -> 2
Other:
- board text added: "TODO: - opi is placed in no-place border region... - SMBJ16CA is bidirectional? - LDO could be smaller - C26 must be 0805 - the simtray filters are 0805 instead of 0603 - forgot to purchase 45R"
- board text added: "prototype. not for consumer use https://devguard.io artanis v0.2 | 2019 | aep"
- board text removed: "prototype not for sale v 0.2 | 2019 | aep"
