File: base/0.3.sch (KiCad schematic (older format))
At the start: 80 parts, among them CON1 MSATA-PCIE_MINI-CARD-MM60-52B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, J1 Conn_02x12_Top_Bottom, J2 SIM_Card, K1 G5Q-1A, K2 G5Q-1A, K3 G5Q-1A, Q1 Q_NPN_BEC, Q2 Q_NPN_BEC, Q3 Q_NPN_BEC, U1 orange_pi_zero, U2 MCP25625-x-SS, U3 OKI-78SR-5_1.5-W36-C, U4 MCP25625-x-SS, U5 LD1085D2M33R, U7 MMA8452Q, Y1 M8AIG-16-12-2T3, Y2 M8AIG-16-12-2T3

Commit message: m
Parts:
- C22, C23, C24: footprint Capacitors:0805 -> Capacitors:0603
- C26: footprint Capacitor_SMD:C_0603_1608Metric -> Capacitor_SMD:C_0805_2012Metric_Pad1.15x1.40mm_HandSolder
- U2, U4: symbol Interface_CAN_LIN:MCP25625-x-SS -> aep:MCP25625-QFN
Connections:
- wire segments 373 -> 374
- no-connect marks 12 -> 68
Other:
- moved on the sheet: C26
Changed lines of the file:
@@
 $EndDescr
-$Comp
-L orangepi-zero:orange_pi_zero U1
-U 1 1 5D6F927A
-P 18150 11350
-F 0 "U1" H 18100 13293 60  0000 C CNN
-F 1 "orange_pi_zero" H 18100 13187 60  0000 C CNN
-F 2 "orangepi-zero:orangepi-zero" H 18100 13081 60  0000 C CNN
-F 3 "" H 17900 12150 60  0000 C CNN
-	1    18150 11350
-	1    0    0    -1
-$EndComp
 $Comp
 L Device:C C7
@@
 Wire Wire Line
 	3100 8850 3100 9100
-Wire Wire Line
-	7600 9550 6600 9550
-Wire Wire Line
-	6950 8150 6600 8150
 NoConn ~ 6600 8850
 NoConn ~ 6600 8750
@@
 F 3 "~" H 6850 9050 50  0001 C CNN
 	1    6850 9050
-	0    -1   -1   0
-$EndComp
-Wire Wire Line
-	6700 9050 6600 9050
+	0    1    1    0
+$EndComp
 Wire Wire Line
 	5400 8350 5250 8350
@@
 Text GLabel 7600 9350 2    118  Input ~ 0
 MISO
-Wire Wire Line
-	6600 9350 7600 9350
 Text GLabel 7050 9450 2    118  Input ~ 0
 MOSI
 Text GLabel 7600 9550 2    118  Input ~ 0
 SCLK
-Wire Wire Line
-	7050 9250 6600 9250
 Text GLabel 6950 8150 2    118  Input ~ 0
 CAN1IRQ
 Wire Wire Line
-	7150 9050 7000 9050
-Wire Wire Line
 	5400 9350 5200 9350
 Wire Wire Line
 	5100 9450 5400 9450
-Wire Wire Line
-	6600 9450 7050 9450
-$Comp
-L Interface_CAN_LIN:MCP25625-x-SS U2
+$Comp
+L aep:MCP25625-QFN U2
 U 1 1 5D895DF1
 P 6000 8850
@@
 Text GLabel 7150 8850 1    118  Input ~ 0
 3.3V
-Wire Wire Line
-	7150 8850 7150 9050
 $Comp
 L Device:C C17
@@
 	3050 12900 3050 13150
 Wire Wire Line
-	7550 13600 6550 13600
-Wire Wire Line
 	6900 12200 6550 12200
 NoConn ~ 6550 12900
@@
 $EndComp
 Wire Wire Line
-	6650 13100 6550 13100
-Wire Wire Line
 	5350 12400 5200 12400
 Wire Wire Line
@@
 Text GLabel 7550 13400 2    118  Input ~ 0
 MISO
-Wire Wire Line
-	6550 13400 7550 13400
 Text GLabel 7000 13500 2    118  Input ~ 0
 MOSI
@@
 Wire Wire Line
 	5050 13500 5350 13500
-Wire Wire Line
-	6550 13500 7000 13500
-$Comp
-L Interface_CAN_LIN:MCP25625-x-SS U4
+$Comp
+L aep:MCP25625-QFN U4
 U 1 1 5D9EF1ED
 P 5950 12900
@@
 	19150 10250 19300 10250
 Connection ~ 19300 10250
-Wire Wire Line
-	19300 10250 19300 9550
-Text GLabel 19550 9550 2    118  Input ~ 0
+Text GLabel 19550 9450 2    118  Input ~ 0
 5V
 Wire Wire Line
-	19300 9550 19500 9550
+	19300 9450 19500 9450
 Wire Wire Line
 	19150 11850 20250 11850
@@
 Connection ~ 18200 4400
 Connection ~ 18500 4400
-$Comp
-L Device:CP C9
-U 1 1 5D752FAD
-P 18350 4400
-F 0 "C9" V 18095 4400 50  0000 C CNN
-F 1 "100uF 50V" V 18186 4400 50  0000 C CNN
-F 2 "Capacitors:CPOL-RADIAL-2.5MM-6.5MM" H 18388 4250 50  0001 C CNN
-F 3 "~" H 18350 4400 50  0001 C CNN
-	1    18350 4400
-	0    1    1    0
-$EndComp
 Wire Wire Line
 	18200 4100 18200 4400
@@
 F 0 "C24" H 7065 2596 50  0000 L CNN
 F 1 "33pF" H 7065 2505 50  0000 L CNN
-F 2 "Capacitors:0805" H 6988 2400 50  0001 C CNN
+F 2 "Capacitors:0603" H 6988 2400 50  0001 C CNN
 F 3 "~" H 6950 2550 50  0001 C CNN
 	1    6950 2550
@@
 F 0 "C23" H 6765 2596 50  0000 L CNN
 F 1 "33pF" H 6765 2505 50  0000 L CNN
-F 2 "Capacitors:0805" H 6688 2400 50  0001 C CNN
+F 2 "Capacitors:0603" H 6688 2400 50  0001 C CNN
 F 3 "~" H 6650 2550 50  0001 C CNN
 	1    6650 2550
@@
 F 0 "C22" H 6365 2596 50  0000 L CNN
 F 1 "33pF" H 6365 2505 50  0000 L CNN
-F 2 "Capacitors:0805" H 6288 2400 50  0001 C CNN
+F 2 "Capacitors:0603" H 6288 2400 50  0001 C CNN
 F 3 "~" H 6250 2550 50  0001 C CNN
 	1    6250 2550
@@
 L Device:C C26
 U 1 1 5DDC6091
-P 19500 9700
-F 0 "C26" V 19248 9700 50  0000 C CNN
-F 1 "10uF" V 19339 9700 50  0000 C CNN
-F 2 "Capacitor_SMD:C_0603_1608Metric" H 19538 9550 50  0001 C CNN
-F 3 "~" H 19500 9700 50  0001 C CNN
-	1    19500 9700
-	1    0    0    -1
-$EndComp
-Connection ~ 19500 9550
-Wire Wire Line
-	19500 9550 19550 9550
+P 19500 9600
+F 0 "C26" V 19248 9600 50  0000 C CNN
+F 1 "10uF" V 19339 9600 50  0000 C CNN
+F 2 "Capacitor_SMD:C_0805_2012Metric_Pad1.15x1.40mm_HandSolder" H 19538 9450 50  0001 C CNN
+F 3 "~" H 19500 9600 50  0001 C CNN
+	1    19500 9600
+	1    0    0    -1
+$EndComp
+Connection ~ 19500 9450
+Wire Wire Line
+	19500 9450 19550 9450
 $Comp
 L power:GND #PWR0132
 U 1 1 5DDC8653
-P 19500 9850
-F 0 "#PWR0132" H 19500 9600 50  0001 C CNN
-F 1 "GND" H 19505 9677 50  0000 C CNN
-F 2 "" H 19500 9850 50  0001 C CNN
-F 3 "" H 19500 9850 50  0001 C CNN
-	1    19500 9850
+P 19500 9900
+F 0 "#PWR0132" H 19500 9650 50  0001 C CNN
+F 1 "GND" H 19505 9727 50  0000 C CNN
+F 2 "" H 19500 9900 50  0001 C CNN
+F 3 "" H 19500 9900 50  0001 C CNN
+	1    19500 9900
 	1    0    0    -1
 $EndComp
@@
 Wire Wire Line
 	21300 11750 21450 11750
+$Comp
+L Device:CP C9
+U 1 1 5D752FAD
+P 18350 4400
+F 0 "C9" V 18095 4400 50  0000 C CNN
+F 1 "100uF 50V" V 18186 4400 50  0000 C CNN
+F 2 "Capacitors:CPOL-RADIAL-2.5MM-6.5MM" H 18388 4250 50  0001 C CNN
+F 3 "~" H 18350 4400 50  0001 C CNN
+	1    18350 4400
+	0    1    1    0
+$EndComp
+NoConn ~ 19150 11050
+NoConn ~ 19150 10850
+NoConn ~ 19150 10750
+NoConn ~ 17050 11000
+NoConn ~ 17050 10900
+NoConn ~ 17050 10800
+NoConn ~ 17050 10700
+NoConn ~ 17050 10600
+NoConn ~ 17050 10500
+NoConn ~ 17050 10400
+NoConn ~ 17050 10300
+NoConn ~ 17050 10200
+NoConn ~ 17050 9900
+NoConn ~ 17050 9800
+NoConn ~ 19150 9900
+NoConn ~ 19150 10000
+$Comp
+L orangepi-zero:orange_pi_zero U1
+U 1 1 5D6F927A
+P 18150 11350
+F 0 "U1" H 18100 13293 60  0000 C CNN
+F 1 "orange_pi_zero" H 18100 13187 60  0000 C CNN
+F 2 "orangepi-zero:orangepi-zero" H 18100 13081 60  0000 C CNN
+F 3 "" H 17900 12150 60  0000 C CNN
+	1    18150 11350
+	1    0    0    -1
+$EndComp
+Wire Wire Line
+	19300 9450 19300 10250
+NoConn ~ 2150 4000
+NoConn ~ 2150 3900
+NoConn ~ 2150 3800
+NoConn ~ 2150 3700
+NoConn ~ 2150 3600
+NoConn ~ 2150 3300
+NoConn ~ 2150 3100
+NoConn ~ 2150 3000
+NoConn ~ 2150 2700
+NoConn ~ 2150 2600
+NoConn ~ 2150 2400
+NoConn ~ 2150 2300
+NoConn ~ 2150 2100
+NoConn ~ 2150 2000
+NoConn ~ 2150 1800
+NoConn ~ 2150 1700
+NoConn ~ 2150 1600
+NoConn ~ 2150 1500
+NoConn ~ 4950 1700
+NoConn ~ 4950 2400
+NoConn ~ 4950 2500
+NoConn ~ 4950 2800
+NoConn ~ 4950 2900
+NoConn ~ 4950 3000
+NoConn ~ 4950 3800
+NoConn ~ 15600 3450
+NoConn ~ 15600 3550
+NoConn ~ 15600 3650
+NoConn ~ 15600 3950
+NoConn ~ 15600 4050
+NoConn ~ 15100 4050
+NoConn ~ 15100 3950
+NoConn ~ 15100 3650
+NoConn ~ 15100 3550
+NoConn ~ 15100 3450
+NoConn ~ 15100 3050
+NoConn ~ 15600 3050
+NoConn ~ 6550 13800
+Wire Wire Line
+	6600 8150 6950 8150
+NoConn ~ 6600 9750
+Wire Wire Line
+	6550 13100 6650 13100
+Wire Wire Line
+	6550 13400 7550 13400
+Wire Wire Line
+	6550 13500 7000 13500
+Wire Wire Line
+	6550 13600 7550 13600
+Wire Wire Line
+	6600 9250 7050 9250
+Wire Wire Line
+	6600 9350 7600 9350
+Wire Wire Line
+	6600 9450 7050 9450
+Wire Wire Line
+	6600 9550 7600 9550
+Wire Wire Line
+	6600 9050 6700 9050
+Wire Wire Line
+	7000 9050 7150 9050
+Wire Wire Line
+	7150 9050 7150 8850
+Wire Wire Line
+	19500 9750 19500 9900
+NoConn ~ 19150 9800
 $EndSCHEMATC
